File: MTV5Beta.sch (EAGLE design)
At the start: 99 parts, among them IC1 OPA2365U, IC2 MCP1700-3302, IC3 MCP1700-3302, J1 MICROUSB, J2 SWDPORT, U1 STM32F405RGT6, U2 ADS8330IB, U3 MX66L51235FZ2I-10G

Commit message: Upload files
Upload files
Parts:
- removed IC3: MCP1700-3302, LDO:XC63FPM
- removed JP7: (no value), pinhead:PINHD-1X6
- removed LED1: red, led:LEDCHIP-LED0805
- removed LED2: green, led:LEDCHIP-LED0805
- removed LED3: blue, led:LEDCHIP-LED0805
- removed PB4: PB, switch-misc:PB
- removed S1: 9077-2, switch-misc:9077-2
- removed TP10, TP11, TP12, TP2, TP5, TP6, TP7, TP8, TP9: TPB1,27, testpad:TPB1,27
- added C33, C34, C36, C38, C39, C40, C42, C44: 0.1uF, rcl:C-EUC0603
- added C35, C37, C41, C43: 2.2uF, rcl:C-EUC0603
- added TP13: TPB1,27, testpad:TPB1,27
- added U$1: 3P-SW, EF_Lib:3P-SW
- added U$2, U$3: TPS73433, EF_Lib:TPS73433
- added U$4: REF2033, EF_Lib:REF2033
- added U$5: LED-RGB, EF_Lib:LED-RGB
- C10, C11: value 6.8pF -> 470pF
- C12, C14, C18, C20, C25: value 10uF -> 0.1uF
- C13: value 1uF -> 20pF
- C15: value 0.1uF -> 20pF
- C16, C17: value 0.1uF -> 10uF
- C2: value 1uF -> 10uF
- C22: value 2.2uF -> 6.8pF
- C23: value 1uF -> 6.8pF
- C27, C28: value 0.1uF -> 2.2uF
- C29: value 10uF -> 2.2uF
- C3, C32, C9: value 1uF -> 0.1uF
- C31: value 1uF -> 2.2uF
- C4: value 0.1uF -> 1uF
- C6: value 470pF -> 1uF
- C7: value 470pF -> 10uF
- JP1: device pinhead:PINHD-1X4 -> pinhead:PINHD-2X4
- JP2: device pinhead:PINHD-1X4 -> pinhead:PINHD-1X2
- JP3: device pinhead:PINHD-1X3 -> pinhead:PINHD-1X4
- JP5: device pinhead:PINHD-1X2 -> pinhead:PINHD-1X3
- JP6: device pinhead:PINHD-1X2 -> pinhead:PINHD-1X6
- R10: value 20 -> 10k
- R11, R12, R16, R24: value 100k -> 100
- R13: value 100 -> 10k
- R14: value 220 -> 1M
- R15, R23: value 100 -> 100k
- R17: value 0 -> 100
- R18: value 0 -> 100k
- R19: value 10k -> 100
- R2: value 2k -> 22
- R20: value 1uH -> 100
- R21: device rcl:R-EU_R0603 -> rcl:R-EU_R0805
- R22: value 100k -> 10k
- R26: value 10k -> 1k
- R27, R29: value 470 -> 1k
- R28: value 470 -> 10k
- R4: value 22 -> 2k
- R5: value 2k -> 1k
- R6: value 20 -> 1k
- R7: value 20 -> 50k
- R8: value 10k -> 20
- R9: value 20 -> 1M
- U1: value STM32F405RGT6 -> ADS8330IB; device EF_Lib:STM32F405RGT6 -> EF_Lib:ADS8330IB
- U2: value ADS8330IB -> STM32F405RGT6; device EF_Lib:ADS8330IB -> EF_Lib:STM32F405RGT6
- Z1: value ASE -> Z-4P; device crystal:ASE -> EF_Lib:Z-4P
Connections:
- removed net N$22: R14.1, U1.PA0_WKUP
- removed net N$24: R17.1, TP7.TP, U1.VBAT
- removed net N$28: TP6.TP, U1.PB5
- removed net N$30: TP8.TP, U1.PB4
- removed net N$31: TP9.TP, U1.PB3
- removed net N$32: TP10.TP, U1.PD2
- removed net N$34: TP11.TP, U1.PB10
- removed net N$35: TP12.TP, U1.PB11
- removed net PB1: R23.1, U1.PB1
- new net LDO_EN: R18.2, R19.2, R20.2, R25.2, U2.PC3
- new net N$36: C27.1, U$3.NR
- new net N$37: IC1A.OUT, R11.2, R7.1
- new net N$38: IC1A.+IN, R5.1
- new net N$40: C1.2, R6.2
- new net PA0: R17.1, U2.PA0_WKUP
- new net VBIAS: C41.1, C42.1, R5.2, U$4.VBIAS
- new net VCC_DEV: C28.1, C30.1, C32.1, C39.1, C40.1, JP1.1, JP1.2, JP3.1, JP6.1, R1.2, R28.1, R4.2, RF1.VCC, U$2.OUT, U$5.COM, U1.+VBD, U3.RESET#, U3.VCC, U3.WP#
- new net VREF: C21.2, C43.1, C44.1, U$4.VREF, U1.REF+
- net ADS_CH0: now also C11.1, R12.1, U1.+IN0; no longer C7.1, R10.1, U2.+IN0
- net ADS_CH1: now also C10.1, R11.1, U1.+IN1; no longer C6.1, R9.1, U2.+IN1
- net AD_CONVST: now also U1.CONVST, U2.PB1; no longer U1.PC5, U2.CONVST
- net AD_CS: now also U1.CS/FS, U2.PC4; no longer U1.PA1, U2.CS/FS
- net AD_INT: now also U1.EOC/INT, U2.PC5; no longer U1.PC4, U2.EOC/INT
- net AGND: now also C10.2, C11.2, C17.2, C19.2, C20.2, C21.1, C27.2, C33.2, C37.2, C38.2, C4.1, C41.2, C42.2, C43.2, C44.2, C5.1, C6.1, JP5.3, U$3.GND, U$4.GND, U1.AGND, U1.COM, U1.REF-; no longer C1.1, C13.2, C14.1, C2.1, C3.1, C30.2, C6.2, C7.2, JP3.3, TP5.TP, U1.VSSA, U2.AGND, U2.COM, U2.REF-
- net AVCC: now also C20.1, C33.1, C4.2, C5.2, C6.2, JP5.1, TP13.TP, U$3.OUT, U1.+VA; no longer C1.2, C13.1, C14.2, C2.2, C3.2, C30.1, JP3.1, R18.2, R20.2, TP2.TP, U1.VDDA, U2.+VA
- net BAT_IN: now also R13.1, U2.PB0; no longer R15.1, U1.PB0
- net FLASH_CS: now also R28.2, U2.PB12; no longer R26.2, U1.PB12
- net GND: now also C13.1, C2.2, C24.2, C28.2, C3.2, C30.2, C34.1, C35.2, C36.1, C39.2, C40.2, C7.2, C8.2, JP1.7, JP1.8, JP2.2, JP3.4, JP6.6, R14.1, R15.1, R18.1, R23.1, U$2.GND, U1.BDGND, U2.VSS, U2.VSSA, U2.VSS_1; no longer C10.2, C11.2, C17.2, C19.2, C20.2, C21.2, C24.1, C27.2, C28.1, C4.2, C5.2, IC3.GND, JP1.4, JP2.4, JP5.2, JP7.6, LED1.C, LED2.C, LED3.C, R11.1, R16.1, R19.1, R24.1, U1.VSS, U1.VSS_1, U2.BDGND, Z1.GND
- net I2C1_SCL: now also JP1.3, JP1.4, U2.PB6; no longer JP1.2, U1.PB6
- net I2C1_SDA: now also JP1.5, JP1.6, R4.1, U2.PB7; no longer JP1.3, R2.1, U1.PB7
- net LED_BLUE: now also R26.2, U2.PC2; no longer R27.2, U1.PC2
- net LED_GREEN: now also R29.1, U2.PC1; no longer R28.2, U1.PC1
- net LED_RED: now also R27.2, U2.PC0; no longer R29.2, U1.PC0
- net N$1: now also R22.2, U2.BOOT0; no longer R19.2, U1.BOOT0
- net N$10: now also R25.1, U$4.EN; no longer U1.PH0, Z1.OUT
- net N$11: now also C35.1, U2.VCAP_2; no longer C26.1, U1.VCAP_2
- net N$12: now also JP5.2; no longer JP4.2
- net N$13: now also R12.2, R8.1; no longer R10.2, R7.1
- net N$14: now also C12.1, R13.2, R14.2, R9.1; no longer C9.1, R12.1, R15.2, R16.2
- net N$15: now also R8.2; no longer R7.2
- net N$16: now also C26.1, U$2.NR; no longer JP6.2, S11.S, S12.S
- net N$17: now also JP2.1, U$1.3; no longer JP5.1, S11.P, S12.P
- net N$18: now also C14.1, R16.1; no longer C8.1, R13.1
- net N$19: now also U$5.R; no longer LED1.A
- net N$2: now also R3.1; no longer R4.1
- net N$20: now also C14.2, R15.2, R17.2; no longer C8.2, R11.2, R14.2
- net N$21: now also R26.1, U$5.B; no longer LED2.A, R28.1
- net N$23: now also R29.2, U$5.G; no longer LED3.A, R29.1
- net N$25: now also C22.1, U2.PC14; no longer C10.1, U1.PC14
- net N$26: now also C23.1, U2.PC15; no longer C11.1, U1.PC15
- net N$27: now also R24.2; no longer R22.2
- net N$29: now also R20.1, U$3.EN; no longer PB4.P, R24.2, R25.2
- net N$3: now also R2.1; no longer R3.1
- net N$4: now also C31.1, U2.VCAP_1; no longer C22.1, U1.VCAP_1
- net N$41: now also IC1A.-IN, R6.1, R7.2; no longer R18.1, U2.REF+
- net N$5: now also C15.1, U2.PH0, Z1.IO1; no longer IC1A.OUT, R6.1, R9.2
- net N$6: now also C8.1, R10.1, U2.NRST; no longer C4.1, R8.1, U1.NRST
- net N$7: now also R19.1, U$2.EN; no longer C25.1, C27.1, IC3.OUT, R20.1
- net N$8: now also C13.2, U2.PH1, Z1.IO2; no longer IC1A.-IN, R6.2
- net N$9: now also C1.1, JP4.2; no longer IC1A.+IN, JP3.2
- net NRF_CE: now also U2.PC7; no longer U1.PC7
- net NRF_CS: now also U2.PC6; no longer U1.PC6
- net NRF_INT: now also U2.PC8; no longer U1.PC8
- net PB2: now also R24.1, U2.PB2; no longer R25.1, U1.PB2
- net SPI1_MISO: now also U1.SDO, U2.PA6; no longer U1.PA6, U2.SDO
- net SPI1_MOSI: now also U1.SDI, U2.PA7; no longer U1.PA7, U2.SDI
- net SPI1_SCK: now also U1.SCLK, U2.PA5; no longer U1.PA5, U2.SCLK
- net SPI2_MISO: now also U2.PB14; no longer RF1.MISO, U1.PB14
- net SPI2_MOSI: now also U2.PB15; no longer RF1.MOSI, U1.PB15
- net SPI2_SCK: now also U2.PB13; no longer RF1.SCK, U1.PB13
- net SPI3_MISO: now also JP6.4, RF1.MISO, U2.PC11; no longer JP7.4, U1.PC11
- net SPI3_MOSI: now also JP6.5, RF1.MOSI, U2.PC12; no longer JP7.5, U1.PC12
- net SPI3_NSS: now also JP6.2, U2.PA4; no longer JP7.2, U1.PA4
- net SPI3_SCK: now also JP6.3, RF1.SCK, U2.PC10; no longer JP7.3, U1.PC10
- net SWCLK: now also U2.PA14; no longer U1.PA14
- net SWDIO: now also U2.PA13; no longer U1.PA13
- net UART2_RX: now also JP3.3, U2.PA3; no longer JP2.3, U1.PA3
- net UART2_TX: now also JP3.2, U2.PA2; no longer JP2.2, U1.PA2
- net USB_DM: now also R3.2, U2.PA11; no longer R4.2, U1.PA11
- net USB_DP: now also R2.2, U2.PA12; no longer R3.2, R5.2, U1.PA12
- net VBUS: now also U2.PA9; no longer U1.PA9
- net VCC: now also C24.1, C25.1, C34.2, C36.2, C7.1, C9.1, R10.2, R16.2, U2.VBAT, U2.VDD, U2.VDDA, U2.VDD_1, U2.VDD_2, U2.VDD_3; no longer C16.1, C17.1, C18.1, C19.1, C23.1, C24.2, C28.2, C31.1, C32.1, C5.1, JP1.1, JP2.1, JP7.1, PB4.S, R1.2, R13.2, R17.2, R2.2, R26.1, R5.1, R8.2, RF1.VCC, U1.VDD, U1.VDD_1, U1.VDD_2, U1.VDD_3, U2.+VBD, U3.RESET#, U3.VCC, U3.WP#, Z1.VDD
- net VIN: now also C16.1, C17.1, C18.1, C19.1, C2.1, C3.1, C37.1, C38.1, R9.2, U$1.2, U$2.IN, U$3.IN, U$4.VIN; no longer C12.1, C15.1, C20.1, C21.1, IC3.IN, JP6.1, R12.2
Other:
- note removed: "Push Button"
- moved on the sheet: C1, C10, C11, C12, C13, C14, C15, C16, C17, C18, C19, C2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

Commit message: v1.0 finished
sch ERC OK!
pcb DRC OK!
gerb export OK!
PDF export OK!
need adding BOM
Parts:
- added TP2: TPB1,27, testpad:TPB1,27
Connections:
- net VCC_DEV: now also TP2.TP
Changed lines of the file:
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@@
 <setting verticaltext="up"/>
 </settings>
-<grid distance="0.05" unitdist="inch" unit="inch" style="lines" multiple="1" display="no" altdistance="0.01" altunitdist="inch" altunit="inch"/>
+<grid distance="0.1" unitdist="inch" unit="inch" style="lines" multiple="1" display="no" altdistance="0.01" altunitdist="inch" altunit="inch"/>
 <layers>
 <layer number="1" name="Top" color="4" fill="1" visible="no" active="no"/>
@@
 <part name="U$5" library="EF_Lib" deviceset="LED-RGB" device=""/>
 <part name="JP1" library="pinhead" deviceset="PINHD-2X4" device=""/>
+<part name="TP2" library="testpad" deviceset="TP" device="B1,27"/>
 </parts>
 <sheets>
@@
 <instance part="U$5" gate="G$1" x="391.16" y="195.58"/>
 <instance part="JP1" gate="A" x="25.4" y="152.4"/>
+<instance part="TP2" gate="G$1" x="241.3" y="289.56"/>
 </instances>
 <busses>
@@
 <junction x="251.46" y="287.02"/>
 <label x="254" y="287.02" size="1.778" layer="95"/>
-</segment>
-<segment>
+<pinref part="TP2" gate="G$1" pin="TP"/>
+</segment>
+<segment>
